File: PCB Design/ANTSATPCB.kicad_pcb (KiCad board)
At the start: 2 copper layers, 50 x 50 mm, 2 parts, among them J1 RFPC-SMA28-F

Commit message: Add files via upload
Parts:
- moved J1 0.76 mm to (-0.04, 9.00)

Commit message: Add files via upload
Parts:
- J1: value RFPC-SMA28-F -> PCB.SMAFST.2H.A.HT; footprint ANTSAV1FOOTPRINT:GRADCONN_RFPC-SMA28-F -> ANTSAV1FOOTPRINT:TAOGLAS_PCB.SMAFST.2H.A.HT; moved to B.Cu
- moved J1 1.00 mm to (0.00, 8.00), turned to 180 degrees
Routing:
- net Net-(ANT1-Pad1): track 0.00 -> 4.39 mm
- net GND: vias 76 -> 74
