File: PCB Design/ANTSATPCB.kicad_pcb (KiCad board)
At the start: 2 copper layers, 50 x 50 mm, 2 parts, among them J1 PCB.SMAFST.2H.A.HT

Commit message: Add files via upload
Parts:
- added H1: MountingHole, MountingHole:MountingHole_3.2mm_M3_Pad, F.Cu at (18.0, 18.0)
- added H2: MountingHole, MountingHole:MountingHole_3.2mm_M3_Pad, F.Cu at (18.0, -18.0)
- added H3: MountingHole, MountingHole:MountingHole_3.2mm_M3_Pad, F.Cu at (-18.0, -18.0)
- added H4: MountingHole, MountingHole:MountingHole_3.2mm_M3_Pad, F.Cu at (-18.0, 18.0)
Routing:
- net GND: vias 83 -> 81
Other:
- outline, holes or cut-outs redrawn
- board text added: "ANTS TAOGLAS ANTENNA BOARD"
- board text added: "Designed by An Nguyen"
