File: PCB Design/ANTSATPCB.kicad_sch (KiCad schematic)
At the start: 2 parts, among them J1 RFPC-SMA28-F

Commit message: Add files via upload
Parts:
- removed J1: RFPC-SMA28-F, ANTSAV1FOOTPRINT:GRADCONN_RFPC-SMA28-F, symbol ANTSATV1SYMBOL:RFPC-SMA28-F
- added J1: PCB.SMAFST.2H.A.HT, ANTSAV1FOOTPRINT:TAOGLAS_PCB.SMAFST.2H.A.HT, symbol ANTSATV1SYMBOL:PCB.SMAFST.2H.A.HT
Connections:
- net GND: now also J1.SH1, J1.SH2
- net at ANT1.1: now also J1.SIG

Commit message: Add files via upload
Parts:
- added H1, H2, H3, H4: MountingHole, MountingHole:MountingHole_3.2mm_M3_Pad, symbol Mechanical:MountingHole
